File: USBSwitch/USBSwitch/USBSwitch.kicad_pcb (KiCad board)
At the start: 2 copper layers, 41 x 32 mm, 17 parts, among them J1 Conn_01x01_Female, J2 Conn_01x01_Female, J3 USB_A, J4 USB_B_Micro

Commit message: Fix usb switch top pour
Routing:
- added copper zone on F.Cu, net GND
- removed copper zone on F.Cu, net (none)
Changed lines of the file:
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@@
     )
   )
-  (zone (net 0) (net_name "") (layer F.Cu) (hatch edge 0.508)
+  (zone (net 1) (net_name GND) (layer F.Cu) (hatch edge 0.508)
     (connect_pads yes (clearance 0.2))
     (min_thickness 0.2)
