File: JLink-SKEDD-adapter/Breakout_JLink.kicad_sch (KiCad schematic)
At the start: 5 parts, among them J1 UART_ClientSide, J2 Conn_02x10_Odd_Even, J3 Jitter_Debug_HostSide, J4 Conn_01x06_Female

Commit message: Breakout JLink: rotate SKEDD footprint with correct cable orientation
(the previous version works OK but the silkscreen arrows point the wrong way)
Parts:
- J3: footprint Jitter_Footprints:WR-WST_REDFIT-6-pins_490107670612 -> Jitter_Footprints:WR-WST_REDFIT-6-pins_490107670612-adapter_to_pcb
Changed lines of the file:
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@@
       (effects (font (size 1.27 1.27)) (justify left))
     )
-    (property "Footprint" "Jitter_Footprints:WR-WST_REDFIT-6-pins_490107670612" (id 2) (at 149.86 110.49 0)
+    (property "Footprint" "Jitter_Footprints:WR-WST_REDFIT-6-pins_490107670612-adapter_to_pcb" (id 2) (at 149.86 110.49 0)
       (effects (font (size 1.27 1.27)) hide)
     )
@@
     )
     (path "/06f35d79-701d-4668-99e8-c39281eb6d67"
-      (reference "J3") (unit 1) (value "Jitter_Debug_HostSide") (footprint "Jitter_Footprints:WR-WST_REDFIT-6-pins_490107670612")
+      (reference "J3") (unit 1) (value "Jitter_Debug_HostSide") (footprint "Jitter_Footprints:WR-WST_REDFIT-6-pins_490107670612-adapter_to_pcb")
     )
     (path "/baa5bd86-b184-4ca9-a98a-4eaeb1dcc77e"

Commit message: Breakout JLink: release V2
- inline UART tx resistor to handle conflict if JLink + Blackmagic hosts both connected
- UART rx pullup resistor to avoid noise if target disconnected or in reset
Parts:
- added R1: 100, Resistor_SMD:R_0603_1608Metric, symbol Device:R
- added R2: 10k, Resistor_SMD:R_0603_1608Metric, symbol Device:R
Connections:
- net Rx_JLink: now also R2.2
- net Tx_JLink: now also R1.1; no longer J1.3 (RX_(client)), J3.1 (TX)
- net VCC: now also R2.1
- new net: J1.3 (RX_(client)), J3.1 (TX), R1.2
Other:
- note added: "Pullup to keep Rx idle while client keeps it floating (e.g. in reset)"
- title: Breakout for JLink Base Compact -> JLink - REDfit adapter
- moved on the sheet: J3
