File: BMP-REDFit-adapter/BMP-REDFit-adapter.kicad_sch (KiCad schematic)
At the start: 6 parts, among them J1 Conn_ARM_JTAG_SWD_10, J2 UART_HostSide, J3 Jitter_Debug_HostSide, J4 Conn_01x02_Pin

Commit message: Modernize the adapter boards
This repo contains adapter boards for the Jitter 6-pins REDFit debug
interface to multiple standard programming/debug tools.
Each now renamed to make this clearer (BMP/HSProbe/JLink) and save those
projects as modern Kicad10 designs
Parts:
- J2: value UART_HostSide -> UART_ClientSide; symbol Jitter_Connectors:UART_HostSide -> Jitter_Connectors:UART_ClientSide
- LOGO1, LOGO2: now left out of the parts list
Other:
- title: (none) -> BMP-REDFit adapter
