File: JLink-REDFit-adapter/JLink-REDFit-adapter.kicad_pcb (KiCad board)
At the start: 2 copper layers, 27.4 x 26 mm, 8 parts, among them J1 UART_ClientSide, J2 2x10 female header 2.56mm pit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, J3 Jitter_Debug_HostSide, J4 Conn_01x06_Socket

Commit message: Modernize the adapter boards
This repo contains adapter boards for the Jitter 6-pins REDFit debug
interface to multiple standard programming/debug tools.
Each now renamed to make this clearer (BMP/HSProbe/JLink) and save those
projects as modern Kicad10 designs
Parts:
- J2: value 2x10 female header 2.56mm pitch. With a notch/key on top side -> 2x10 female header 2.54mm pitch. With a notch/key on top side
Connections:
- net /RX_client renamed /to_client
- net /TX_client renamed /from_client
