File: JLink-to-TC2030-IDC__microchip/JLink-to-TC2030-IDC__microchip.kicad_pcb (KiCad board)
At the start: 2 copper layers, 27.4 x 26 mm, 7 parts, among them J1 Conn_02x10_Odd_Even, J2 Conn_02x10_Odd_Even, J3 uart_host_2.54, SW1 Reset

Commit message: Modernize the adapter boards
This repo contains adapter boards for the Jitter 6-pins REDFit debug
interface to multiple standard programming/debug tools.
Each now renamed to make this clearer (BMP/HSProbe/JLink) and save those
projects as modern Kicad10 designs
Other:
- board text added: "JLink to TC2030-IDC Microchip-specific pinout!"
- board text removed: "JLink - TC2030-IDC Microchip-specific pinout!"
