File: SL23-modem-tester/battery_charger.kicad_sch (KiCad schematic)
At the start: 59 parts, among them J11 JST PH 2-pin, J13 61200621621, Q1 CSD17581Q3A, Q2 CSD17581Q3A, Q3 CSD17581Q3A, Q4 CSD17581Q3A, Q5 CSD17581Q3A, Q7 BSS138BK,215, U1 BQ25672

Commit message: SL23: clarify design slightly, add README
Other:
- note removed: "Button and filter is placed on seperate board! Is connected through a header, see page 13."
Changed lines of the file:
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@@
-		)
-	)
-	(text "Button and filter is placed on seperate board! \nIs connected through a header, see page 13."
-		(exclude_from_sim no)
-		(at 102.87 175.26 0)
-		(effects
-			(font
-				(size 1.905 1.905)
-				(italic yes)
-			)
-			(justify left bottom)
-			(href "#13")
 		)
 	)
