File: SL23-modem-tester/SL23-modem-tester.kicad_pcb (KiCad board)
At the start: 4 copper layers, 120 x 107 mm, 229 parts, among them J1 691322310002, J10 Conn_01x30, J12 30320-6002HB, J13 61200621621, J2 MM60-EZH039-B5-R850, J4 68602-450HLF, J5 swd_with_uart_client, J7 ‎MM60-52B1-G1-R850‎, Q1 CSD17581Q3A, Q2 CSD17581Q3A, Q3 CSD17581Q3A, Q4 CSD17581Q3A, Q5 CSD17581Q3A, Q7 BSS138BK,215, SW2 SW_Push, U1 BQ25672, U11 MCP9701A, U2 SIC473ED-T1-GE3, U3 SIC473ED-T1-GE3, U5 STM32L4R7ZITx, U6 SLG59M301V, U8 W25Q256JVEIQ, Y1 12 MHz, Y2 32.768kHz

Commit message: SL23-modem-tester: release after manual review
Routing:
- net GND: vias 360 -> 447
- added copper zone on In2.Cu, net Net-(U1-SW1)
- added copper zone on In2.Cu, net Net-(U1-SW2)
- removed copper zone on B.Cu, net Net-(U1-SW1)
- removed copper zone on B.Cu, net Net-(U1-SW2)
