File: SL23-modem-tester/cellular.kicad_sch (KiCad schematic)
At the start: 13 parts, among them J2 MM60-EZH039-B5-R850, J7 ‎MM60-52B1-G1-R850‎, U6 SLG59M301V

Commit message: SL23-modem-tester: release after manual review
Other:
- note removed: "A bypass capacitor (C3) of no less than 470 μF with low ESR should be used"
- note removed: "Add additional UART to mini PCIe for GPS use? --> Quectel datasheet: Keep all NC, RESERVED and unused pins unconnected. --> COEX1 & COEX1 can be used for additional UART, however, it is in 1V8 domain."
- note removed: "Click to go back to home"
Changed lines of the file:
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@@
 		(effects
 			(font
-				(size 0.5 0.5)
+				(size 0.8 0.8)
 			)
 			(justify right bottom)
-		)
-	)
-	(text "Add additional UART to mini PCIe for GPS use?\n--> Quectel datasheet: Keep all NC, RESERVED and unused pins unconnected.\n--> COEX1 & COEX1 can be used for additional UART, however, it is in 1V8 domain.\n"
-		(exclude_from_sim no)
-		(at 22.86 163.83 0)
-		(effects
-			(font
-				(size 1.27 1.27)
-			)
-			(justify left bottom)
 		)
 	)
@@
 		)
 	)
-	(text "Click to go back to home"
-		(exclude_from_sim no)
-		(at 280.67 22.86 0)
-		(effects
-			(font
-				(size 2.54 2.54)
-				(italic yes)
-			)
-			(justify right bottom)
-			(href "#1")
-		)
-	)
-	(text "A bypass capacitor (C3) of no less than 470 μF with low ESR should be used"
-		(exclude_from_sim no)
-		(at 24.13 97.79 0)
-		(effects
-			(font
-				(size 1.27 1.27)
-			)
-			(justify left bottom)
-		)
-	)
