File: SL23-modem-tester/storage.kicad_sch (KiCad schematic)
At the start: 5 parts, among them U8 W25Q256JVEIQ

Commit message: SL23-modem-tester: release after manual review
Other:
- note removed: "(NOR-flash, 512M-bit, 4Kb Uniform Sector)"
- note removed: "(for prototype 256M-bit version is used!)"
Changed lines of the file:
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@@
 		(rev "1")
-	)
-	(text "(NOR-flash, 512M-bit, 4Kb Uniform Sector)"
-		(exclude_from_sim no)
-		(at 33.02 20.32 0)
-		(effects
-			(font
-				(size 1.905 1.905)
-			)
-			(justify left bottom)
-		)
 	)
 	(text "SPI flash"
@@
 			)
 			(justify left bottom)
-		)
-	)
-	(text "(for prototype 256M-bit version is used!)"
-		(exclude_from_sim no)
-		(at 33.02 24.13 0)
-		(effects
-			(font
-				(size 1.905 1.905)
-			)
-			(justify left bottom)
